Commit message: Update 9 Oct

File: oscbf/assets/mycobot/mycobot_urdf_grip.urdf (robot description, URDF)
Before this commit: robot firefighter, 7 links, 6 joints
Links:
- added link gripper_base, mass 0.05; collision mesh filename=mycobot_adaptive_gripper/gripper_base.dae; visual mesh filename=mycobot_adaptive_gripper/gripper_base.dae
- added link gripper_left1, mass 0.01; collision mesh filename=mycobot_adaptive_gripper/gripper_left1.dae; visual mesh filename=mycobot_adaptive_gripper/gripper_left1.dae
- added link gripper_left2, mass 0.01; collision mesh filename=mycobot_adaptive_gripper/gripper_left2.dae; visual mesh filename=mycobot_adaptive_gripper/gripper_left2.dae
- added link gripper_left3, mass 0.01; collision mesh filename=mycobot_adaptive_gripper/gripper_left3.dae; visual mesh filename=mycobot_adaptive_gripper/gripper_left3.dae
- added link gripper_right1, mass 0.01; collision mesh filename=mycobot_adaptive_gripper/gripper_right1.dae; visual mesh filename=mycobot_adaptive_gripper/gripper_right1.dae
- added link gripper_right2, mass 0.01; collision mesh filename=mycobot_adaptive_gripper/gripper_right2.dae; visual mesh filename=mycobot_adaptive_gripper/gripper_right2.dae
- added link gripper_right3, mass 0.01; collision mesh filename=mycobot_adaptive_gripper/gripper_right3.dae; visual mesh filename=mycobot_adaptive_gripper/gripper_right3.dae
Joints:
- added joint gripper_base_to_gripper_left2: type revolute, parent gripper_base, child gripper_left2, origin xyz=-0.005 0.027 0 rpy=0 0 0, axis 0 0 1, limit lower=-0.8 upper=0.5 effort=1000.0 velocity=0, mimic joint=gripper_controller multiplier=1.0 offset=0
- added joint gripper_base_to_gripper_right2: type revolute, parent gripper_base, child gripper_right2, origin xyz=0.005 0.027 0 rpy=0 0 0, axis 0 0 1, limit lower=-0.5 upper=0.8 effort=1000.0 velocity=0, mimic joint=gripper_controller multiplier=-1.0 offset=0
- added joint gripper_base_to_gripper_right3: type revolute, parent gripper_base, child gripper_right3, origin xyz=0.012 0.005 0 rpy=0 0 0, axis 0 0 1, limit lower=-0.15 upper=0.7 effort=1000.0 velocity=0, mimic joint=gripper_controller multiplier=-1.0 offset=0
- added joint gripper_controller: type revolute, parent gripper_base, child gripper_left3, origin xyz=-0.012 0.005 0 rpy=0 0 0, axis 0 0 1, limit lower=-0.74 upper=0.15 effort=1000.0 velocity=0
- added joint gripper_left3_to_gripper_left1: type revolute, parent gripper_left3, child gripper_left1, origin xyz=-0.027 0.016 0 rpy=0 0 0, axis 0 0 1, limit lower=-0.5 upper=0.5 effort=1000.0 velocity=0, mimic joint=gripper_controller multiplier=-1.0 offset=0
- added joint gripper_right3_to_gripper_right1: type revolute, parent gripper_right3, child gripper_right1, origin xyz=0.027 0.016 0 rpy=0 0 0, axis 0 0 1, limit lower=-0.5 upper=0.5 effort=1000.0 velocity=0, mimic joint=gripper_controller multiplier=1.0 offset=0
- added joint gripper_to_flange_joint: type fixed, parent joint6_flange, child gripper_base, origin xyz=0 0 0 rpy=0 0 0
